Commit message: initial commit

File: ar_description/urdf/ar.ros2_control.xacro (robot description, xacro)
@@ -22,6 +22,6 @@
       <joint name="joint_1">
         <command_interface name="position">
-          <param name="min">${robot_parameters['j1_limit_min']}</param>
-          <param name="max">${robot_parameters['j1_limit_max']}</param>
+          <param name="min">{-170*pi/180}</param>
+          <param name="max">{170*pi/180}</param>
         </command_interface>
         <state_interface name="position">
@@ -32,6 +32,6 @@
       <joint name="joint_2">
         <command_interface name="position">
-          <param name="min">${robot_parameters['j2_limit_min']}</param>
-          <param name="max">${robot_parameters['j2_limit_max']}</param>
+          <param name="min">{-42*pi/180}</param>
+          <param name="max">{90*pi/180}</param>
         </command_interface>
         <state_interface name="position">
@@ -42,6 +42,6 @@
       <joint name="joint_3">
         <command_interface name="position">
-          <param name="min">${robot_parameters['j3_limit_min']}</param>
-          <param name="max">${robot_parameters['j3_limit_max']}</param>
+          <param name="min">{-89*pi/180}</param>
+          <param name="max">{52*pi/180}</param>
         </command_interface>
         <state_interface name="position">
@@ -52,6 +52,6 @@
       <joint name="joint_4">
         <command_interface name="position">
-          <param name="min">${robot_parameters['j4_limit_min']}</param>
-          <param name="max">${robot_parameters['j4_limit_max']}</param>
+          <param name="min">${-robot_parameters['j4_limit']}</param>
+          <param name="max">${robot_parameters['j4_limit']}</param>
         </command_interface>
         <state_interface name="position">
@@ -62,6 +62,6 @@
       <joint name="joint_5">
         <command_interface name="position">
-          <param name="min">${robot_parameters['j5_limit_min']}</param>
-          <param name="max">${robot_parameters['j5_limit_max']}</param>
+          <param name="min">{-105*pi/180}</param>
+          <param name="max">{105*pi/180}</param>
         </command_interface>
         <state_interface name="position">
@@ -72,6 +72,6 @@
       <joint name="joint_6">
         <command_interface name="position">
-          <param name="min">${robot_parameters['j6_limit_min']}</param>
-          <param name="max">${robot_parameters['j6_limit_max']}</param>
+          <param name="min">${-robot_parameters['j6_limit']}</param>
+          <param name="max">${robot_parameters['j6_limit']}</param>
         </command_interface>
         <state_interface name="position">

File: ar_description/urdf/ar_gripper.ros2_control.xacro (robot description, xacro)
@@ -23,4 +23,5 @@
         <param name="mimic">gripper_jaw1_joint</param>
         <param name="multiplier">1</param>
+        <command_interface name="position" />
         <state_interface name="position">
           <param name="initial_value">0.0</param>

File: ar_description/urdf/ar_macro.xacro (robot description, xacro)
@@ -61,5 +61,5 @@
       <child link="link_1"/>
       <axis xyz="0 0 1"/>
-      <limit lower="${robot_parameters['j1_limit_min']}" upper="${robot_parameters['j1_limit_max']}" effort="0" velocity="0.5"/>
+      <limit lower="${-170.0 / 180.0 * pi}" upper="${170.0 / 180.0 * pi}" effort="0" velocity="0.5"/>
     </joint>
     <link name="link_2">
@@ -90,5 +90,5 @@
       <child link="link_2"/>
       <axis xyz="0 0 -1"/>
-      <limit lower="${robot_parameters['j2_limit_min']}" upper="${robot_parameters['j2_limit_max']}" effort="0.5" velocity="0.5"/>
+      <limit lower="${-42.0 / 180.0 * pi}" upper="${90.0 / 180.0 * pi}" effort="0.5" velocity="0.5"/>
     </joint>
     <link name="link_3">
@@ -119,5 +119,5 @@
       <child link="link_3"/>
       <axis xyz="0 0 -1"/>
-      <limit lower="${robot_parameters['j3_limit_min']}" upper="${robot_parameters['j3_limit_max']}" effort="0" velocity="0.5"/>
+      <limit lower="${-89.0 / 180.0 * pi}" upper="${52.0 / 180.0 * pi}" effort="0" velocity="0.5"/>
     </joint>
     <link name="link_4">
@@ -148,5 +148,5 @@
       <child link="link_4"/>
       <axis xyz="0 0 -1"/>
-      <limit lower="${robot_parameters['j4_limit_min']}" upper="${robot_parameters['j4_limit_max']}" effort="0" velocity="0.5"/>
+      <limit lower="${-1 * robot_parameters['j4_limit']}" upper="${robot_parameters['j4_limit']}" effort="0" velocity="0.5"/>
     </joint>
     <link name="link_5">
@@ -177,5 +177,5 @@
       <child link="link_5"/>
       <axis xyz="1 0 0"/>
-      <limit lower="${robot_parameters['j5_limit_min']}" upper="${robot_parameters['j5_limit_max']}" effort="0" velocity="1.0"/>
+      <limit lower="${-105.0 / 180.0 * pi}" upper="${105.0 / 180.0 * pi}" effort="0" velocity="1.0"/>
     </joint>
     <link name="link_6">
@@ -206,5 +206,5 @@
       <child link="link_6"/>
       <axis xyz="0 0 1"/>
-      <limit lower="${robot_parameters['j6_limit_min']}" upper="${robot_parameters['j6_limit_max']}" effort="0" velocity="1.0"/>
+      <limit lower="${-1.0 * robot_parameters['j6_limit']}" upper="${robot_parameters['j6_limit']}" effort="0" velocity="1.0"/>
     </joint>
     <!-- center of the end effector mounting surface on link_6 -->
